File: DesignAssignments/FINALDAkicadpcb/FINALDAkicadpcb.kicad_pcb (KiCad board)
At the start: 2 copper layers, 24 parts, among them J1 Conn_01x02_Pin, J2 Conn_01x03_Pin, J3 Conn_01x04_Socket, J4 Conn_01x08, J5 Conn_01x10, J6 Conn_01x06, J7 Conn_01x06, J8 Conn_01x08, U2 TB6612FNG, U3 CC56-12SRWA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

Commit message: Signed-off-by: CaFu0320 <jeff20674@gmail.com>
Parts:
- moved J7 96.8 mm to (90.0, 79.5)
- moved J1 89.2 mm to (90.0, 103.2)
- moved S1 87.3 mm to (119.0, 96.0)
- moved J6 85.4 mm to (90.0, 58.5)
- moved U2 83.3 mm to (106.0, 95.5)
- moved J8 78.6 mm to (90.0, 31.5)
- moved U3 78.1 mm to (119.3, 122.0), turned to 90 degrees
- moved S2 73.6 mm to (131.5, 96.0)
- moved R4 50.6 mm to (143.0, 94.5)
- moved J3 50.4 mm to (162.0, 104.7)
- moved R3 40.5 mm to (142.0, 86.0)
- moved J2 29.1 mm to (162.0, 89.6)
- moved J4 25.7 mm to (162.0, 63.8)
- moved J5 7.76 mm to (162.0, 31.0)
- moved R1 5.41 mm to (120.5, 82.0)
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Routing:
- net 3V3: track 0.00 -> 247.3 mm, vias 0 -> 3
- net GND: track 0.00 -> 233.5 mm, vias 0 -> 4
- net PD2: track 0.00 -> 166.7 mm, vias 0 -> 2
- net PD3: track 0.00 -> 116.8 mm, vias 0 -> 4
- net PC4: track 0.00 -> 113.6 mm, vias 0 -> 1
- net PC5: track 0.00 -> 108.9 mm, vias 0 -> 1
- net PD1: track 0.00 -> 94.6 mm, vias 0 -> 2
- net PB5: track 0.00 -> 81.1 mm, vias 0 -> 2
- net PB4: track 0.00 -> 66.5 mm, vias 0 -> 1
- net Net-(U3-CC1): track 0.00 -> 65.8 mm, vias 0 -> 1
- net PD6: track 0.00 -> 65.6 mm, vias 0 -> 1
- net PD5: track 0.00 -> 65.3 mm, vias 0 -> 1
- net Net-(U3-a): track 0.00 -> 63.0 mm, vias 0 -> 2
- net PC0: track 0.00 -> 62.3 mm, vias 0 -> 1
- net PB3: track 0.00 -> 58.3 mm, vias 0 -> 1
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Other:
- board outline added: 92 x 110.5 mm
