File: DesignAssignments/FINALDAkicadpcb/FINALDAkicadpcb.kicad_sch (KiCad schematic)
At the start: 24 parts, among them J1 Conn_01x02_Pin, J2 Conn_01x03_Pin, J3 Conn_01x04_Socket, J4 Conn_01x08, J5 Conn_01x10, J6 Conn_01x06, J7 Conn_01x06, J8 Conn_01x08, U2 TB6612FNG, U3 CC56-12SRWA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

Commit message: Signed-off-by: CaFu0320 <jeff20674@gmail.com>
Other:
- note added: "7-SEG DISPLAY"
- note added: "BMI 160 CUSTOM CHIP"
- note added: "DC MOTOR CONNECTIONS"
- note added: "LED'S"
- note added: "MOTOR DRIVER"
- note added: "OLED"
- note added: "PINS"
- note added: "POTENTIOMETER"
- note added: "PUSH BUTTONS"
- note added: "SERVO MOTOR CONNECTIONS"
- note added: "ULTRASONIC SENSOR CONNECTORS"
- moved on the sheet: C1, D1, D2, DS1, J1, J2, J3, R1, R2, U1, U2, U3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
